File: hw/keyboardv2.kicad_pcb (KiCad board)
At the start: 2 copper layers, 145 x 45 mm, 43 parts, among them K1 CONN_4, K2 CONN_4, K3 CONN_4, K4 CONN_4, K5 CONN_4, K6 CONN_4, K7 CONN_4, K8 CONN_4, Q1 MOSFET_N, U1 TINYMEGA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

Commit message: Assign LED resistor values, change some labels for readability
Parts:
- added MARKER: VAL**, MARKER, F.Cu at (217.2, 106.5)
- R1: value R -> 180
- R10, R3, R4, R5, R6, R7, R8, R9: value R -> 270
- R2: value R -> 220
Other:
- board size 145 x 45 mm -> 112 x 45.5 mm
Changed lines of the file:
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@@
     (links 140)
     (no_connects 0)
-    (area 74.949999 99.949999 221.545001 145.050001)
+    (area 107.949999 99.949999 220.050001 145.550001)
     (thickness 1.6)
     (drawings 5)
     (tracks 966)
     (zones 0)
-    (modules 43)
+    (modules 44)
     (nets 72)
   )
@@
   )
   (setup
-    (last_trace_width 1)
+    (last_trace_width 0.25)
     (user_trace_width 0.25)
     (user_trace_width 0.4)
@@
     (pad_to_mask_clearance 0)
     (aux_axis_origin 75 100)
-    (visible_elements 7FFFFF8F)
+    (visible_elements 7FFFFFBF)
     (pcbplotparams
       (layerselection 3178497)
@@
       (effects (font (size 0.50038 0.4572) (thickness 0.1143)) (justify mirror))
     )
-    (fp_text value R (at -1.69926 0 360) (layer B.SilkS)
+    (fp_text value 180 (at -1.69926 0 360) (layer B.SilkS)
       (effects (font (size 0.508 0.4572) (thickness 0.1143)) (justify mirror))
     )
@@
       (effects (font (size 0.50038 0.4572) (thickness 0.1143)) (justify mirror))
     )
-    (fp_text value R (at -1.69926 0 360) (layer B.SilkS)
+    (fp_text value 270 (at -1.69926 0 360) (layer B.SilkS)
       (effects (font (size 0.508 0.4572) (thickness 0.1143)) (justify mirror))
     )
@@
       (effects (font (size 0.50038 0.4572) (thickness 0.1143)) (justify mirror))
     )
-    (fp_text value R (at -1.69926 0 360) (layer B.SilkS)
+    (fp_text value 270 (at -1.69926 0 360) (layer B.SilkS)
       (effects (font (size 0.508 0.4572) (thickness 0.1143)) (justify mirror))
     )
@@
       (effects (font (size 0.50038 0.4572) (thickness 0.1143)) (justify mirror))
     )
-    (fp_text value R (at -1.69926 0 360) (layer B.SilkS)
+    (fp_text value 270 (at -1.69926 0 360) (layer B.SilkS)
       (effects (font (size 0.508 0.4572) (thickness 0.1143)) (justify mirror))
     )
@@
       (effects (font (size 0.50038 0.4572) (thickness 0.1143)) (justify mirror))
     )
-    (fp_text value R (at -1.69926 0 360) (layer B.SilkS)
+    (fp_text value 270 (at -1.69926 0 360) (layer B.SilkS)
       (effects (font (size 0.508 0.4572) (thickness 0.1143)) (justify mirror))
     )
@@
       (effects (font (size 0.50038 0.4572) (thickness 0.1143)))
     )
-    (fp_text value R (at -1.69926 0 360) (layer F.SilkS)
+    (fp_text value 220 (at -1.69926 0 360) (layer F.SilkS)
       (effects (font (size 0.508 0.4572) (thickness 0.1143)))
     )
@@
       (effects (font (size 0.50038 0.4572) (thickness 0.1143)) (justify mirror))
     )
-    (fp_text value R (at -1.69926 0 360) (layer B.SilkS)
+    (fp_text value 270 (at -1.69926 0 360) (layer B.SilkS)
       (effects (font (size 0.508 0.4572) (thickness 0.1143)) (justify mirror))
     )
@@
       (effects (font (size 0.50038 0.4572) (thickness 0.1143)) (justify mirror))
     )
-    (fp_text value R (at -1.69926 0 360) (layer B.SilkS)
+    (fp_text value 270 (at -1.69926 0 360) (layer B.SilkS)
       (effects (font (size 0.508 0.4572) (thickness 0.1143)) (justify mirror))
     )
@@
       (effects (font (size 0.50038 0.4572) (thickness 0.1143)) (justify mirror))
     )
-    (fp_text value R (at -1.69926 0 360) (layer B.SilkS)
+    (fp_text value 270 (at -1.69926 0 360) (layer B.SilkS)
       (effects (font (size 0.508 0.4572) (thickness 0.1143)) (justify mirror))
     )
@@
       (effects (font (size 0.50038 0.4572) (thickness 0.1143)) (justify mirror))
     )
-    (fp_text value R (at -1.69926 0 360) (layer B.SilkS)
+    (fp_text value 270 (at -1.69926 0 360) (layer B.SilkS)
       (effects (font (size 0.508 0.4572) (thickness 0.1143)) (justify mirror))
     )
@@
     )
   )
+  (module MARKER (layer F.Cu)
+    (at 217.25 106.5)
+    (fp_text reference MARKER (at 0 -1.27) (layer F.SilkS)
+      (effects (font (size 1 1) (thickness 0.15)))
+    )
+    (fp_text value VAL** (at 0 1.27) (layer F.SilkS)
+      (effects (font (size 1 1) (thickness 0.15)))
+    )
+    (pad ~ thru_hole circle (at 0 0) (size 1.397 1.397) (drill 0.8128)
+      (layers *.Cu *.Mask F.SilkS)
+    )
+  )
+  (gr_line (start 108 100) (end 108 145.5) (angle 90) (layer Edge.Cuts) (width 0.1))
+  (gr_line (start 220 145.5) (end 220 100) (angle 90) (layer Edge.Cuts) (width 0.1))
+  (gr_line (start 108 145.5) (end 220 145.5) (angle 90) (layer Edge.Cuts) (width 0.1))
+  (gr_line (start 108 100) (end 220 100) (angle 90) (layer Edge.Cuts) (width 0.1))
   (gr_circle (center 96.8 123) (end 96.8 133) (layer Dwgs.User) (width 0.2))
-  (gr_line (start 220 100) (end 75 100) (angle 90) (layer Edge.Cuts) (width 0.1))
-  (gr_line (start 220 145) (end 220 100) (angle 90) (layer Edge.Cuts) (width 0.1))
-  (gr_line (start 75 145) (end 220 145) (angle 90) (layer Edge.Cuts) (width 0.1))
-  (gr_line (start 75 100) (end 75 145) (angle 90) (layer Edge.Cuts) (width 0.1))
   (segment (start 202.08 141.33) (end 201.585 140.835) (width 0.25) (layer B.Cu) (net 1))
   (segment (start 194.6 132.3) (end 195.87 131.03) (width 0.25) (layer B.Cu) (net 1))
